File: pe/charles-leong-buhconverter-kicad/charlesleong.kicad_pcb (KiCad board)
At the start: 2 copper layers, 9 parts, among them U1 TPS542025DDCR

Commit message: pre-shower progress
Parts:
- moved C3 2.83 mm to (111.0, 64.0)
- moved C7 2.12 mm to (117.9, 81.5)
- moved C1 2.12 mm to (110.5, 70.5)
- moved L1 2.06 mm to (110.5, 79.0)
- moved C2 1.58 mm to (118.0, 66.0)
- moved C4 1.56 mm to (117.9, 77.5)
- moved C6 1.12 mm to (125.0, 70.5)
- moved C5 1.00 mm to (125.0, 79.5)
- moved U1 1.00 mm to (118.0, 73.0)
Routing:
- added copper zone on B.Cu, net GND
Other:
- board outline added: 25 x 25 mm
Changed lines of the file:
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@@
 		(capping no)
 		(filling no)
-		(zone_defaults)
 		(pcbplotparams
 			(layerselection 0x00000000_00000000_55555555_5755f5ff)
@@
 	(footprint "Capacitor_SMD:C_2220_5750Metric_Pad1.97x5.40mm_HandSolder"
 		(layer "F.Cu")
-		(at 126 71 90)
+		(at 125 70.5 90)
 		(descr "Capacitor SMD 2220 (5750 Metric), square (rectangular) end terminal, IPC-7351 nominal with elongated pad for handsoldering. (Body size from: http://datasheets.avx.com/AVX-HV_MLCC.pdf)")
 		(tags "capacitor handsolder")
@@
 	(footprint "Capacitor_SMD:C_1210_3225Metric_Pad1.33x2.70mm_HandSolder"
 		(layer "F.Cu")
-		(at 120 82)
+		(at 117.9375 81.5)
 		(descr "Capacitor SMD 1210 (3225 Metric), square (rectangular) end terminal, IPC-7351 nominal with elongated pad for handsoldering. (Body size source: IPC-SM-782 page 76, https://www.pcb-3d.com/wordpress/wp-content/uploads/ipc-sm-782a_amendment_1_and_2.pdf)")
 		(tags "capacitor handsolder")
@@
 	(footprint "Package_TO_SOT_SMD:SOT-23-6"
 		(layer "F.Cu")
-		(at 119 73)
+		(at 118 73)
 		(descr "SOT, 6 Pin (JEDEC MO-178 Var AB https://www.jedec.org/document_search?search_api_views_fulltext=MO-178)")
 		(tags "SOT TO_SOT_SMD")
@@
 	(footprint "Capacitor_SMD:C_1210_3225Metric_Pad1.33x2.70mm_HandSolder"
 		(layer "F.Cu")
-		(at 119.5 77.5)
+		(at 117.9375 77.5)
 		(descr "Capacitor SMD 1210 (3225 Metric), square (rectangular) end terminal, IPC-7351 nominal with elongated pad for handsoldering. (Body size source: IPC-SM-782 page 76, https://www.pcb-3d.com/wordpress/wp-content/uploads/ipc-sm-782a_amendment_1_and_2.pdf)")
 		(tags "capacitor handsolder")
@@
 	(footprint "Capacitor_SMD:C_2220_5750Metric_Pad1.97x5.40mm_HandSolder"
 		(layer "F.Cu")
-		(at 126 79.5 -90)
+		(at 125 79.5 -90)
 		(descr "Capacitor SMD 2220 (5750 Metric), square (rectangular) end terminal, IPC-7351 nominal with elongated pad for handsoldering. (Body size from: http://datasheets.avx.com/AVX-HV_MLCC.pdf)")
 		(tags "capacitor handsolder")
@@
 		)
 		(property "Value" "10μf"
-			(at 0 3.65 90)
+			(at 1 3.7125 90)
 			(layer "F.Fab")
 			(effects
@@
 	(footprint "formula_slug_footprint_library:L_Wurth_WE-PD2SR-7850"
 		(layer "F.Cu")
-		(at 112.5 79.5 90)
+		(at 110.5 79 90)
 		(descr "Shielded Power Inductor, body 7.8x7x5mm, https://www.we-online.com/en/components/products/WE-PD2SR#/articles/WE-PD2SR-7850")
 		(tags "SMT")
@@
 	(footprint "Capacitor_SMD:C_2220_5750Metric_Pad1.97x5.40mm_HandSolder"
 		(layer "F.Cu")
-		(at 119.5 66.5 90)
+		(at 118 66 90)
 		(descr "Capacitor SMD 2220 (5750 Metric), square (rectangular) end terminal, IPC-7351 nominal with elongated pad for handsoldering. (Body size from: http://datasheets.avx.com/AVX-HV_MLCC.pdf)")
 		(tags "capacitor handsolder")
@@
 	(footprint "Capacitor_SMD:C_2220_5750Metric_Pad1.97x5.40mm_HandSolder"
 		(layer "F.Cu")
-		(at 112 72)
+		(at 110.5 70.5)
 		(descr "Capacitor SMD 2220 (5750 Metric), square (rectangular) end terminal, IPC-7351 nominal with elongated pad for handsoldering. (Body size from: http://datasheets.avx.com/AVX-HV_MLCC.pdf)")
 		(tags "capacitor handsolder")
@@
 	(footprint "Capacitor_SMD:C_1210_3225Metric_Pad1.33x2.70mm_HandSolder"
 		(layer "F.Cu")
-		(at 113 66)
+		(at 111 64)
 		(descr "Capacitor SMD 1210 (3225 Metric), square (rectangular) end terminal, IPC-7351 nominal with elongated pad for handsoldering. (Body size source: IPC-SM-782 page 76, https://www.pcb-3d.com/wordpress/wp-content/uploads/ipc-sm-782a_amendment_1_and_2.pdf)")
 		(tags "capacitor handsolder")
@@
 			)
 		)
+	)
+	(gr_rect
+		(start 105 60)
+		(end 130 85)
+		(stroke
+			(width 0.0508)
+			(type default)
+		)
+		(fill no)
+		(layer "Edge.Cuts")
+	)
+	(zone
+		(net "GND")
+		(layer "B.Cu")
+		(name "GND")
+		(hatch edge 0.5)
+		(connect_pads
+			(clearance 0.508)
+		)
+		(min_thickness 0.25)
+		(fill yes
+			(thermal_gap 0.5)
+			(thermal_bridge_width 0.5)
+			(island_removal_mode 0)
+		)
+		(polygon
+			(pts
+				(xy 105.5 84.5) (xy 105.5 60.5) (xy 129.5 60.5) (xy 129.5 84.5)
+			)
+		)

Commit message: I lied i didn't shower, pre-shower pcb updates
Parts:
- moved C3 1.58 mm to (111.5, 65.5), turned to 180 degrees
- moved L1 1.58 mm to (112.0, 78.5)
- moved C4 1.17 mm to (119.0, 77.0), turned to 180 degrees
- moved C7 1.17 mm to (119.0, 81.0)
- moved C2 1.12 mm to (118.5, 67.0)
- moved C5 1.00 mm to (125.0, 78.5)
- moved U1 1.00 mm to (119.0, 73.0)
- moved C1 0.50 mm to (111.0, 70.5), turned to 180 degrees
- moved C6 0.50 mm to (125.0, 70.0)
Routing:
- net Net-(U1-SW): track 0.00 -> 26.2 mm
- net +5V: track 0.00 -> 21.2 mm
- net +15V: track 0.00 -> 16.1 mm
- net GND: track 0.00 -> 10.7 mm, vias 0 -> 5
- net Net-(U1-BOOT): track 0.00 -> 5.95 mm
Other:
- board size 25 x 25 mm -> 25 x 24 mm

Commit message: i will not shower until then
Parts:
- turned L1 to -90 degrees
Routing:
- net Net-(U1-SW): track 26.2 -> 13.0 mm
- net +5V: track 21.2 -> 19.4 mm
Changed lines of the file:
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@@
 	(footprint "formula_slug_footprint_library:L_Wurth_WE-PD2SR-7850"
 		(layer "F.Cu")
-		(at 112 78.5 90)
+		(at 112 78.5 -90)
 		(descr "Shielded Power Inductor, body 7.8x7x5mm, https://www.we-online.com/en/components/products/WE-PD2SR#/articles/WE-PD2SR-7850")
 		(tags "SMT")
 		(property "Reference" "L1"
-			(at 0 -5 90)
+			(at 0 -5 270)
 			(unlocked yes)
 			(layer "F.SilkS")
@@
 		)
 		(property "Value" "12 µH"
-			(at 0 5 90)
+			(at 0 5 270)
 			(unlocked yes)
 			(layer "F.Fab")
@@
 		)
 		(property "Digikey Part Number" "732-4529-6-ND"
-			(at 0 0 90)
+			(at 0 0 270)
 			(unlocked yes)
 			(layer "F.Fab")
@@
 		)
 		(property "Digikey URL" "https://www.digikey.com/en/products/detail/w%C3%BCrth-elektronik/744787120/4155880"
-			(at 0 0 90)
+			(at 0 0 270)
 			(unlocked yes)
 			(layer "F.Fab")
@@
 		)
 		(property "Manufacturer" "Würth Elektronik"
-			(at 0 0 90)
+			(at 0 0 270)
 			(unlocked yes)
 			(layer "F.Fab")
@@
 		)
 		(property "Manufacturer Part Number" "744787120"
-			(at 0 0 90)
+			(at 0 0 270)
 			(unlocked yes)
 			(layer "F.Fab")
@@
 		(duplicate_pad_numbers_are_jumpers no)
 		(fp_line
+			(start -3.9 4.01)
+			(end 3.9 4.01)
+			(stroke
+				(width 0.12)
+				(type solid)
+			)
+			(layer "F.SilkS")
+		)
+		(fp_line
 			(start 0 -4.01)
 			(end 3.9 -4.01)
-			(stroke
-				(width 0.12)
-				(type solid)
-			)
-			(layer "F.SilkS")
-		)
-		(fp_line
-			(start -3.9 4.01)
-			(end 3.9 4.01)
 			(stroke
 				(width 0.12)
@@
 		)
 		(fp_line
+			(start -1.95 3.5)
+			(end 1.95 3.5)
+			(stroke
+				(width 0.1)
+				(type solid)
+			)
+			(layer "F.Fab")
+		)
+		(fp_line
 			(start -1.95 -3.5)
 			(end 1.95 -3.5)
@@
 			(layer "F.Fab")
 		)
-		(fp_line
+		(fp_arc
 			(start -1.95 3.5)
-			(end 1.95 3.5)
+			(mid -3.9 0)
+			(end -1.95 -3.5)
 			(stroke
 				(width 0.1)
@@
 			(layer "F.Fab")
 		)
-		(fp_arc
-			(start -1.95 3.5)
-			(mid -3.9 0)
-			(end -1.95 -3.5)
-			(stroke
-				(width 0.1)
-				(type solid)
-			)
-			(layer "F.Fab")
-		)
 		(fp_text user "${REFERENCE}"
-			(at 0 0 90)
+			(at 0 0 270)
 			(unlocked yes)
 			(layer "F.Fab")
@@
 		)
 		(pad "1" smd rect
-			(at -2.5 0 90)
+			(at -2.5 0 270)
 			(size 3 7.5)
 			(layers "F.Cu" "F.Mask" "F.Paste")
@@
 		)
 		(pad "2" smd rect
-			(at 2.5 0 90)
+			(at 2.5 0 270)
 			(size 3 7.5)
 			(layers "F.Cu" "F.Mask" "F.Paste")
@@
 	)
 	(segment
-		(start 113.7875 76)
-		(end 117.4375 79.65)
+		(start 117.4375 81)
+		(end 112 81)
 		(width 0.254)
 		(layer "F.Cu")
@@
 	)
 	(segment
-		(start 117.4375 79.65)
-		(end 117.4375 81)
-		(width 0.254)
-		(layer "F.Cu")
-		(net "+5V")
-	)
-	(segment
 		(start 121.5935 79.269)
 		(end 119.1685 79.269)
@@
 	)
 	(segment
-		(start 112 76)
-		(end 113.7875 76)
+		(start 110.988 81)
+		(end 112 81)
 		(width 0.254)
 		(layer "F.Cu")
@@
 	)
 	(segment
-		(start 107.869 74.119)
-		(end 107.869 77.881)
-		(width 0.254)
-		(layer "F.Cu")
-		(net "Net-(U1-SW)")
-	)
-	(segment
-		(start 116.131 74.119)
-		(end 107.869 74.119)
-		(width 0.254)
-		(layer "F.Cu")
-		(net "Net-(U1-SW)")
-	)
-	(segment
-		(start 107.869 77.881)
-		(end 110.988 81)
+		(start 113 77)
+		(end 112 76)
 		(width 0.254)
 		(layer "F.Cu")
@@
 	)
 	(segment
+		(start 117.4375 77)
+		(end 113 77)
+		(width 0.254)
+		(layer "F.Cu")
+		(net "Net-(U1-SW)")
+	)
+	(segment
 		(start 118.906 75.5315)
 		(end 117.4375 77)
@@
 	)
 	(segment
-		(start 117.4375 77)
-		(end 117.4375 75.4255)
-		(width 0.254)
-		(layer "F.Cu")
-		(net "Net-(U1-SW)")
-	)
-	(segment
-		(start 117.4375 75.4255)
-		(end 116.131 74.119)
-		(width 0.254)
-		(layer "F.Cu")
-		(net "Net-(U1-SW)")
-	)
-	(segment
-		(start 110.988 81)
-		(end 112 81)
-		(width 0.254)
-		(layer "F.Cu")
+		(start 112 76)
+		(end 113.7875 76)
+		(width 0.254)
+		(layer "F.Cu")

Commit message: 11:24pm
Routing:
- net GND: track 10.7 -> 15.2 mm, vias 5 -> 8
Changed lines of the file:
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@@
+	)
+	(segment
+		(start 117.8625 72.05)
+		(end 116.55 72.05)
+		(width 0.254)
+		(layer "F.Cu")
+		(net "GND")
 	)
 	(segment
 		(start 122 64.3625)
 		(end 118.5 64.3625)
+		(width 0.254)
+		(layer "F.Cu")
+		(net "GND")
+	)
+	(segment
+		(start 120.1375 74.8625)
+		(end 120 75)
 		(width 0.254)
 		(layer "F.Cu")
@@
 	)
 	(segment
+		(start 120.5625 82.9375)
+		(end 120.5 83)
+		(width 0.254)
+		(layer "F.Cu")
+		(net "GND")
+	)
+	(segment
 		(start 108.3625 70.5)
 		(end 106.5 70.5)
@@
 	)
 	(segment
+		(start 120.5625 81)
+		(end 120.5625 82.9375)
+		(width 0.254)
+		(layer "F.Cu")
+		(net "GND")
+	)
+	(segment
+		(start 116.55 72.05)
+		(end 116.5 72)
+		(width 0.254)
+		(layer "F.Cu")
+		(net "GND")
+	)
+	(segment
 		(start 108.5 70.5)
 		(end 108.3625 70.5)
+		(width 0.254)
+		(layer "F.Cu")
+		(net "GND")
+	)
+	(segment
+		(start 120.1375 73.95)
+		(end 120.1375 74.8625)
 		(width 0.254)
 		(layer "F.Cu")
@@
 	)
 	(via
+		(at 120.5 83)
+		(size 0.508)
+		(drill 0.254)
+		(layers "F.Cu" "B.Cu")
+		(net "GND")
+	)
+	(via
 		(at 108.5 65.5)
 		(size 0.508)
@@
 		(size 0.508)
 		(drill 0.254)
+		(layers "F.Cu" "B.Cu")
+		(net "GND")
+	)
+	(via
+		(at 120 75)
+		(size 0.508)
+		(drill 0.254)
+		(layers "F.Cu" "B.Cu")
+		(net "GND")
+	)
+	(via
+		(at 116.5 72)
+		(size 0.508)
+		(drill 0.254)

Commit message: 11:32 pm.
Parts:
- moved C1 25.0 mm to (131.0, 85.5)
- moved C2 25.0 mm to (138.5, 82.0)
- moved C3 25.0 mm to (131.5, 80.5)
- moved C4 25.0 mm to (139.0, 92.0)
- moved C5 25.0 mm to (145.0, 93.5)
- moved C6 25.0 mm to (145.0, 85.0)
- moved C7 25.0 mm to (139.0, 96.0)
- moved L1 25.0 mm to (132.0, 93.5)
- moved U1 25.0 mm to (139.0, 88.0)

Commit message: DRC settled
Parts:
- moved C5 1.12 mm to (146.0, 94.0)
- moved C7 0.71 mm to (139.5, 96.5)
Routing:
- net +5V: track 19.4 -> 22.1 mm
Changed lines of the file:
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@@
 		(tags "capacitor handsolder")
 		(property "Reference" "C6"
-			(at 0 -3.65 90)
+			(at 4.5 1.5 180)
 			(layer "F.SilkS")
 			(effects
@@
 	(footprint "Capacitor_SMD:C_1210_3225Metric_Pad1.33x2.70mm_HandSolder"
 		(layer "F.Cu")
-		(at 139 96)
+		(at 139.5 96.5)
 		(descr "Capacitor SMD 1210 (3225 Metric), square (rectangular) end terminal, IPC-7351 nominal with elongated pad for handsoldering. (Body size source: IPC-SM-782 page 76, https://www.pcb-3d.com/wordpress/wp-content/uploads/ipc-sm-782a_amendment_1_and_2.pdf)")
 		(tags "capacitor handsolder")
 		(property "Reference" "C7"
-			(at 0 -2.3 0)
+			(at 0 2.5 0)
 			(layer "F.SilkS")
 			(effects
@@
 		(tags "SOT TO_SOT_SMD")
 		(property "Reference" "U1"
-			(at 0 -2.4 0)
+			(at -3 0 0)
 			(layer "F.SilkS")
 			(effects
@@
 		(tags "capacitor handsolder")
 		(property "Reference" "C4"
-			(at 0 -2.3 0)
+			(at 2 -2.5 0)
 			(layer "F.SilkS")
 			(effects
@@
 	(footprint "Capacitor_SMD:C_2220_5750Metric_Pad1.97x5.40mm_HandSolder"
 		(layer "F.Cu")
-		(at 145 93.5 -90)
+		(at 146 94 -90)
 		(descr "Capacitor SMD 2220 (5750 Metric), square (rectangular) end terminal, IPC-7351 nominal with elongated pad for handsoldering. (Body size from: http://datasheets.avx.com/AVX-HV_MLCC.pdf)")
 		(tags "capacitor handsolder")
 		(property "Reference" "C5"
-			(at 0 -3.65 90)
+			(at -4.5 -0.5 180)
 			(layer "F.SilkS")
 			(effects
@@
 		(tags "SMT")
 		(property "Reference" "L1"
-			(at 0 -5 270)
+			(at 0 5 0)
 			(unlocked yes)
 			(layer "F.SilkS")
@@
 		(tags "capacitor handsolder")
 		(property "Reference" "C2"
-			(at 0 -3.65 90)
+			(at 4.5 -0.5 180)
 			(layer "F.SilkS")
 			(effects
@@
 		(tags "capacitor handsolder")
 		(property "Reference" "C1"
-			(at 0 -3.65 0)
+			(at 4.5 1 0)
 			(layer "F.SilkS")
 			(effects
@@
 		(tags "capacitor handsolder")
 		(property "Reference" "C3"
-			(at 0 -2.3 0)
+			(at 0 2.5 0)
 			(layer "F.SilkS")
 			(effects
@@
 	)
 	(segment
-		(start 145 90.8625)
+		(start 137.9375 96.5)
+		(end 137.4375 96)
+		(width 0.254)
+		(layer "F.Cu")
+		(net "+5V")
+	)
+	(segment
+		(start 145 90.3625)
 		(end 145 87.6375)
 		(width 0.254)
@@
 	)
 	(segment
-		(start 145 90.8625)
-		(end 141.5935 94.269)
+		(start 146 91.3625)
+		(end 145 90.3625)
 		(width 0.254)
 		(layer "F.Cu")
@@
 	)
 	(segment
-		(start 139.1685 94.269)
-		(end 137.4375 96)
+		(start 137.9375 95.5)
+		(end 137.9375 96.5)
 		(width 0.254)
 		(layer "F.Cu")
@@
 	)
 	(segment
-		(start 141.5935 94.269)
-		(end 139.1685 94.269)
+		(start 143.3625 94)
+		(end 139.4375 94)
+		(width 0.254)
+		(layer "F.Cu")
+		(net "+5V")
+	)
+	(segment
+		(start 139.4375 94)
+		(end 137.9375 95.5)
 		(width 0.254)
 		(layer "F.Cu")
@@
 	)
 	(segment
+		(start 146 91.3625)
+		(end 143.3625 94)
+		(width 0.254)
+		(layer "F.Cu")
+		(net "+5V")
+	)
+	(segment
 		(start 137.8625 87.05)
 		(end 136.55 87.05)
+		(width 0.254)
+		(layer "F.Cu")
+		(net "GND")
+	)
+	(segment
+		(start 141.0625 96.5)
+		(end 140.5625 97)
 		(width 0.254)
 		(layer "F.Cu")
@@
 	)
 	(segment
+		(start 146 96.6375)
+		(end 145 97.6375)
+		(width 0.254)
+		(layer "F.Cu")
+		(net "GND")
+	)
+	(segment
 		(start 129.9375 80.5)
 		(end 128.5 80.5)
@@
 	)
 	(segment
-		(start 140.5625 97.9375)
-		(end 140.5 98)
+		(start 141.0625 96.5)
+		(end 142.5 96.5)
 		(width 0.254)
 		(layer "F.Cu")
@@
 	)
 	(segment
-		(start 145 96.1375)
+		(start 145 97.6375)
 		(end 145 98)
-		(width 0.254)
-		(layer "F.Cu")
-		(net "GND")
-	)
-	(segment
-		(start 140.5625 96)
-		(end 140.5625 97.9375)
 		(width 0.254)
 		(layer "F.Cu")
@@
 	)
 	(via
-		(at 140.5 98)
+		(at 142.5 96.5)
 		(size 0.508)
 		(drill 0.254)
